Commit message: Update commit

File: install/testbot/share/testbot/description/test_robot.urdf.xacro (robot description, xacro)
@@ -2,4 +2,5 @@
 <robot name="test_robot" xmlns:xacro="http://www.ros.org/wiki/xacro">
     <xacro:include filename="test_robot_core.xacro" />
-    <xacro:include filename="ros2_control.xacro" />
+    <!-- <xacro:include filename="ros2_control.xacro" /> -->
+    <xacro:include filename="lidar.xacro" />
 </robot>

File: install/testbot/share/testbot/description/test_robot_core.xacro (robot description, xacro)
@@ -36,5 +36,5 @@
     </link>
     <!-- LIDAR LINK -->
-    <link name="lidar">
+    <link name="lidar_module">
         <visual>
             <geometry>
@@ -116,7 +116,7 @@
     </joint>
     <!-- LIDAR JOINT -->
-    <joint name="base_lidar_joint" type="fixed">
+    <joint name="base_lidar_module_joint" type="fixed">
         <parent link="base_link" />
-        <child link="lidar" />
+        <child link="lidar_module" />
         <origin xyz="0 0 0.225" rpy="0 0 0" />
     </joint>
