Commit message: Update

File: install/testbot/share/testbot/description/test_robot_core.xacro (robot description, xacro)
@@ -62,5 +62,6 @@
         <collision>
             <geometry>
-                <cylinder radius ="0.1" length="0.05" />
+                <!-- use sphere collider for minimal contact with ground to eliminate wheel drift -->
+                <sphere radius ="0.1" />
             </geometry>
             <origin xyz="0 0.025 0" rpy="1.57 0 0" />
@@ -81,5 +82,6 @@
         <collision>
             <geometry>
-                <cylinder radius="0.1" length="0.05" />
+                <!-- use sphere colliders for minimal contact with ground to eliminate wheel drift -->
+                <sphere radius="0.1" />
             </geometry>
             <origin xyz="0 -0.025 0" rpy="-1.57 0 0" />
@@ -108,4 +110,8 @@
         </xacro:inertial_sphere>
     </link>
+    <gazebo reference="caster_wheel">
+        <mu1 value ="0.001"/>
+        <mu2 value ="0.001"/>
+    </gazebo>
 #JOINTS
     <!-- ROBOT BODY FOOTPRINT JOINT -->
