Commit message: Update

File: install/testbot/share/testbot/description/inertial_macros.xacro (robot description, xacro)
@@ -1,32 +1 @@
-<?xml version="1.0"?>
-<robot xmlns:xacro="http://www.ros.org/wiki/xacro" >
-    <!-- Specify some standard inertial calculations https://en.wikipedia.org/wiki/List_of_moments_of_inertia -->
-    <!-- These make use of xacro's mathematical functionality -->
-    <xacro:macro name="inertial_sphere" params="mass radius *origin">
-        <inertial>
-            <xacro:insert_block name="origin"/>
-            <mass value="${mass}" />
-            <inertia ixx="${(2/5) * mass * (radius*radius)}" ixy="0.0" ixz="0.0"
-                    iyy="${(2/5) * mass * (radius*radius)}" iyz="0.0"
-                    izz="${(2/5) * mass * (radius*radius)}" />
-        </inertial>
-    </xacro:macro>
-    <xacro:macro name="inertial_box" params="mass x y z *origin">
-        <inertial>
-            <xacro:insert_block name="origin"/>
-            <mass value="${mass}" />
-            <inertia ixx="${(1/12) * mass * (y*y+z*z)}" ixy="0.0" ixz="0.0"
-                    iyy="${(1/12) * mass * (x*x+z*z)}" iyz="0.0"
-                    izz="${(1/12) * mass * (x*x+y*y)}" />
-        </inertial>
-    </xacro:macro>
-    <xacro:macro name="inertial_cylinder" params="mass radius length *origin">
-        <inertial>
-            <xacro:insert_block name="origin"/>
-            <mass value="${mass}" />
-            <inertia ixx="${(1/12) * mass * (3*radius*radius + length*length)}" ixy="0.0" ixz="0.0"
-                    iyy="${(1/12) * mass * (3*radius*radius + length*length)}" iyz="0.0"
-                    izz="${(1/2) * mass * (radius*radius)}" />
-        </inertial>
-    </xacro:macro>
-</robot>
+/home/rae/testbot_ws/src/testbot/description/inertial_macros.xacro

File: install/testbot/share/testbot/description/lidar.xacro (robot description, xacro)
@@ -1,54 +1 @@
-<?xml version="1.0"?>
-<robot xmlns:xacro="http://www.ros.org/wiki/xacro">
-    <link name="lidar_link">
-        <visual>
-            <geometry>
-                <cylinder radius="0.09" length="0.05" />
-            </geometry>
-            <origin xyz="0 0 0" rpy="0 0 0" />
-            <material name="white" />
-        </visual>
-        <collision>
-            <geometry>
-                <box size ="0.18 0.18 0.05" />
-            </geometry>
-            <origin xyz="0 0 0" rpy="0 0 0" />
-        </collision>
-    </link>
-    <joint name="base_laser_joint" type="fixed">
-        <parent link="base_link"/>
-        <child link="lidar_link"/>
-        <origin xyz="0 0 0.225" rpy="0 0 0"/>
-    </joint>
-    <gazebo reference="lidar_link">
-        <sensor name="lidar_sensor" type="gpu_lidar">
-            <topic>LaserScan</topic>
-            <pose>0 0 0 0 0 0</pose>
-            <update_rate>10</update_rate>
-            <ray>
-                <scan>
-                    <horizontal>
-                        <samples>360</samples>
-                        <resolution>1</resolution>
-                        <min_angle>-3.14</min_angle>
-                        <max_angle>3.14</max_angle>
-                    </horizontal>
-                </scan>
-                <range>
-                    <min>0.3</min>
-                    <max>12</max>
-                    <resolution>0.01</resolution>
-                </range>
-            </ray>
-            <always_on>1</always_on>
-            <visualize>true</visualize>
-        </sensor>
-    </gazebo>
-    <gazebo>
-        <plugin
-            filename="libignition-gazebo-sensors-system.so"
-            name="ignition::gazebo::systems::Sensors">
-            <render_engine>ogre2</render_engine>
-        </plugin>
-    </gazebo>
-</robot>
+/home/rae/testbot_ws/src/testbot/description/lidar.xacro

File: install/testbot/share/testbot/description/ros2_control.xacro (robot description, xacro)
@@ -1,32 +1 @@
-<?xml version="1.0"?>
-<robot xmlns:xacro="http://www.ros.org/wiki/xacro">
-    <ros2_control name="GazeboSimControl" type="system">
-        <hardware>
-            <plugin>ign_ros2_control/GazeboSimControl</plugin>
-        </hardware>
-        <joint name="base_left_wheel_joint">
-            <command_interface name="velocity">
-                <param name="min">-10 </param>
-                <param name="max">10 </param>
-            </command_interface>
-            <state_interface name ="velocity"/>
-            <state_interface name ="position"/>
-        </joint>
-        <joint name="base_right_wheel_joint">
-            <command_interface name="velocity">
-                <param name="min">-10 </param>
-                <param name="max">10 </param>
-            </command_interface>
-            <state_interface name ="velocity"/>
-            <state_interface name ="position"/>
-        </joint>
-    </ros2_control>
-    <gazebo>
-        <plugin filename="libign_ros2_control-system.so" name="ign_ros2_control">
-            <robot_param>robot_description</robot_param>
-            <robot_param_node>robot_state_publisher</robot_param_node>
-            <parameters>$(find testbot)/config/controllers.yaml</parameters>
-            <controller_manager_prefix_node_name>controller_manager</controller_manager_prefix_node_name>
-        </plugin>
-    </gazebo>
-</robot>
+/home/rae/testbot_ws/src/testbot/description/ros2_control.xacro

File: install/testbot/share/testbot/description/test_robot.urdf.xacro (robot description, xacro)
@@ -1,6 +1 @@
-<?xml version="1.0"?>
-<robot name="test_robot" xmlns:xacro="http://www.ros.org/wiki/xacro">
-    <xacro:include filename="test_robot_core.xacro" />
-    <xacro:include filename="ros2_control.xacro" />
-    <xacro:include filename="lidar.xacro" />
-</robot>
+/home/rae/testbot_ws/src/testbot/description/test_robot.urdf.xacro

File: install/testbot/share/testbot/description/test_robot_core.xacro (robot description, xacro)
@@ -1,149 +1 @@
-<?xml version="1.0"?>
-<robot xmlns:xacro="http://www.ros.org/wiki/xacro">
-#Include connected files
-    <xacro:include filename="inertial_macros.xacro" />
-#Define colours
-    <material name="grey">
-        <color rgba="0.5 0.5 0.5 1" />
-    </material>
-    <material name="purple">
-        <color rgba="0.8 0 0.7 1" />
-    </material>
-    <material name="white">
-        <color rgba ="1 1 1 1" />
-    </material>
-#LINKS
-    <!-- ROBOT FOOTPRINT LINK -->
-    <link name="base_footprint" />
-    <!-- ROBOT BODY LINK -->
-    <link name="base_link">
-        <visual>
-            <geometry>
-                <box size ="0.6 0.4 0.2" />
-            </geometry>
-            <origin xyz="0 0 0.1" rpy="0 0 0" />
-            <material name="purple" />
-        </visual>
-        <collision>
-            <geometry>
-                <box size ="0.6 0.4 0.2" />
-            </geometry>
-            <origin xyz="0 0 0.1" rpy="0 0 0" />
-        </collision>
-        <xacro:inertial_box mass="0.5" x="0.6" y="0.4" z="0.2">
-            <origin xyz="0 0 0.1" rpy="0 0 0" />
-        </xacro:inertial_box>
-    </link>
-    <!-- LIDAR LINK -->
-    <link name="lidar_module">
-        <visual>
-            <geometry>
-                <cylinder radius="0.09" length="0.05" />
-            </geometry>
-            <origin xyz="0 0 0" rpy="0 0 0" />
-            <material name="white" />
-        </visual>
-        <collision>
-            <geometry>
-                <box size ="0.18 0.18 0.05" />
-            </geometry>
-            <origin xyz="0 0 0" rpy="0 0 0" />
-        </collision>
-    </link>
-    <!-- LEFT WHEEL LINK -->
-    <link name="left_wheel">
-        <visual>
-            <geometry>
-                <cylinder radius="0.1" length="0.05" />
-            </geometry>
-            <origin xyz="0 0.025 0" rpy="1.57 0 0" />
-            <material name="grey" />
-        </visual>
-        <collision>
-            <geometry>
-                <!-- use sphere collider for minimal contact with ground to eliminate wheel drift -->
-                <sphere radius ="0.1" />
-            </geometry>
-            <origin xyz="0 0.025 0" rpy="1.57 0 0" />
-        </collision>
-        <xacro:inertial_cylinder mass="0.1" radius="0.1" length="0.05">
-            <origin xyz="0 0.025 0" rpy="1.57 0 0" />
-        </xacro:inertial_cylinder>
-    </link>
-    <!-- RIGHT WHEEL LINK -->
-    <link name="right_wheel">
-        <visual>
-            <geometry>
-                <cylinder radius="0.1" length="0.05" />
-            </geometry>
-            <origin xyz="0 -0.025 0" rpy="-1.57 0 0" />
-            <material name="grey" />
-        </visual>
-        <collision>
-            <geometry>
-                <!-- use sphere colliders for minimal contact with ground to eliminate wheel drift -->
-                <sphere radius="0.1" />
-            </geometry>
-            <origin xyz="0 -0.025 0" rpy="-1.57 0 0" />
-        </collision>
-        <xacro:inertial_cylinder mass="0.1" radius="0.1" length="0.05">
-            <origin xyz="0 -0.025 0" rpy="-1.57 0 0" />
-        </xacro:inertial_cylinder>
-    </link>
-    <!-- CASTER WHEEL LINK -->
-    <link name="caster_wheel">
-        <visual>
-            <geometry>
-                <sphere radius="0.05" />
-            </geometry>
-            <origin xyz="0 0 -0.05" rpy="0 0 0" />
-            <material name="grey" />
-        </visual>
-        <collision>
-            <geometry>
-                <sphere radius="0.05" />
-            </geometry>
-            <origin xyz="0 0 -0.05" rpy="0 0 0" />
-        </collision>
-        <xacro:inertial_sphere mass="0.08" radius="0.05">
-            <origin xyz="0 0 -0.05" rpy="0 0 0" />
-        </xacro:inertial_sphere>
-    </link>
-    <gazebo reference="caster_wheel">
-        <mu1 value ="0.001"/>
-        <mu2 value ="0.001"/>
-    </gazebo>
-#JOINTS
-    <!-- ROBOT BODY FOOTPRINT JOINT -->
-    <joint name="base_joint" type="fixed">
-        <parent link="base_footprint" />
-        <child link="base_link" />
-        <origin xyz="0 0 0.1" rpy="0 0 0" />
-    </joint>
-    <!-- LIDAR JOINT -->
-    <joint name="base_lidar_module_joint" type="fixed">
-        <parent link="base_link" />
-        <child link="lidar_module" />
-        <origin xyz="0 0 0.225" rpy="0 0 0" />
-    </joint>
-    <!-- LEFT WHEEL JOINT -->
-    <joint name="base_left_wheel_joint" type="continuous">
-        <parent link="base_link" />
-        <child link="left_wheel" />
-        <origin xyz="-0.15 0.2 0" rpy="0 0 0" />
-        <axis xyz="0 1 0" />
-    </joint>
-    <!-- RIGHT WHEEL JOINT -->
-    <joint name="base_right_wheel_joint" type="continuous">
-        <parent link="base_link" />
-        <child link="right_wheel" />
-        <origin xyz="-0.15 -0.2 0" rpy="0 0 0" />
-        <axis xyz="0 1 0" />
-    </joint>
-    <!-- CASTER WHEEL JOINT -->
-    <joint name="base_caster_wheel_joint" type="fixed">
-        <parent link="base_link" />
-        <child link="caster_wheel" />
-        <origin xyz="0.2 0 0" rpy="0 0 0" />
-    </joint>
-</robot>
+/home/rae/testbot_ws/src/testbot/description/test_robot_core.xacro

File: src/testbot/description/ros2_control.xacro (robot description, xacro)
@@ -1,32 +1,3 @@
 <?xml version="1.0"?>
 <robot xmlns:xacro="http://www.ros.org/wiki/xacro">
-    <ros2_control name="GazeboSimControl" type="system">
-        <hardware>
-            <plugin>ign_ros2_control/GazeboSimControl</plugin>
-        </hardware>
-        <joint name="base_left_wheel_joint">
-            <command_interface name="velocity">
-                <param name="min">-10 </param>
-                <param name="max">10 </param>
-            </command_interface>
-            <state_interface name ="velocity"/>
-            <state_interface name ="position"/>
-        </joint>
-        <joint name="base_right_wheel_joint">
-            <command_interface name="velocity">
-                <param name="min">-10 </param>
-                <param name="max">10 </param>
-            </command_interface>
-            <state_interface name ="velocity"/>
-            <state_interface name ="position"/>
-        </joint>
-    </ros2_control>
-    <gazebo>
-        <plugin filename="libign_ros2_control-system.so" name="ign_ros2_control">
-            <robot_param>robot_description</robot_param>
-            <robot_param_node>robot_state_publisher</robot_param_node>
-            <parameters>$(find testbot)/config/controllers.yaml</parameters>
-            <controller_manager_prefix_node_name>controller_manager</controller_manager_prefix_node_name>
-        </plugin>
-    </gazebo>
 </robot>

File: src/testbot/description/test_robot.urdf.xacro (robot description, xacro)
@@ -2,5 +2,5 @@
 <robot name="test_robot" xmlns:xacro="http://www.ros.org/wiki/xacro">
     <xacro:include filename="test_robot_core.xacro" />
-    <xacro:include filename="ros2_control.xacro" />
+    <!-- <xacro:include filename="ros2_control.xacro" /> -->
     <xacro:include filename="lidar.xacro" />
 </robot>

File: src/testbot/description/test_robot_core.xacro (robot description, xacro)
@@ -147,3 +147,31 @@
         <origin xyz="0.2 0 0" rpy="0 0 0" />
     </joint>
+    <ros2_control name="IgnitionSystem" type="system">
+        <hardware>
+            <plugin>ign_ros2_control/IgnitionSystem</plugin>
+        </hardware>
+        <joint name="base_left_wheel_joint">
+            <command_interface name="velocity">
+                <param name="min">-10 </param>
+                <param name="max">10 </param>
+            </command_interface>
+            <state_interface name ="velocity"/>
+            <state_interface name ="position"/>
+        </joint>
+        <joint name="base_right_wheel_joint">
+            <command_interface name="velocity">
+                <param name="min">-10 </param>
+                <param name="max">10 </param>
+            </command_interface>
+            <state_interface name ="velocity"/>
+            <state_interface name ="position"/>
+        </joint>
+    </ros2_control>
+    <gazebo>
+        <plugin filename="libign_ros2_control-system.so" name="ign_ros2_control::IgnitionROS2ControlPlugin">
+            <robot_param>robot_description</robot_param>
+            <robot_param_node>robot_state_publisher</robot_param_node>
+            <parameters>$(find testbot)/config/controllers.yaml</parameters>
+        </plugin>
+    </gazebo>
 </robot>
