Commit message: Update push

File: src/testbot/description/lidar.xacro (robot description, xacro)
@@ -1,4 +1,5 @@
 <?xml version="1.0"?>
 <robot xmlns:xacro="http://www.ros.org/wiki/xacro">
+    <!-- INITIATE GAZEBO LIDAR SENSOR -->
     <link name="lidar_link">
         <visual>
@@ -25,5 +26,5 @@
             <topic>LaserScan</topic>
             <pose>0 0 0 0 0 0</pose>
-            <update_rate>10</update_rate>
+            <update_rate>5</update_rate>
             <ray>
                 <scan>

File: src/testbot/description/ros2_control.xacro (robot description, xacro)
@@ -1,3 +1,31 @@
 <?xml version="1.0"?>
 <robot xmlns:xacro="http://www.ros.org/wiki/xacro">
+    <ros2_control name="IgnitionSystem" type="system">
+        <hardware>
+            <plugin>ign_ros2_control/IgnitionSystem</plugin>
+        </hardware>
+        <joint name="base_left_wheel_joint">
+            <command_interface name="velocity">
+                <param name="min">-10 </param>
+                <param name="max">10 </param>
+            </command_interface>
+            <state_interface name ="velocity"/>
+            <state_interface name ="position"/>
+        </joint>
+        <joint name="base_right_wheel_joint">
+            <command_interface name="velocity">
+                <param name="min">-10 </param>
+                <param name="max">10 </param>
+            </command_interface>
+            <state_interface name ="velocity"/>
+            <state_interface name ="position"/>
+        </joint>
+    </ros2_control>
+    <gazebo>
+        <plugin filename="ign_ros2_control-system" name="ign_ros2_control::IgnitionROS2ControlPlugin">
+            <robot_param>robot_description</robot_param>
+            <robot_param_node>robot_state_publisher</robot_param_node>
+            <parameters>$(find testbot)/config/controllers.yaml</parameters>
+        </plugin>
+    </gazebo>
 </robot>

File: src/testbot/description/test_robot.urdf.xacro (robot description, xacro)
@@ -3,4 +3,5 @@
     <xacro:include filename="test_robot_core.xacro" />
     <!-- <xacro:include filename="ros2_control.xacro" /> -->
+    <xacro:include filename="gazebo_control.xacro" />
     <xacro:include filename="lidar.xacro" />
 </robot>
