Commit message: Update

File: src/testbot/description/gazebo_control.xacro (robot description, xacro)
@@ -4,34 +4,30 @@
         <plugin name="ignition::gazebo::systems::DiffDrive" filename="ignition-gazebo-diff-drive-system">
             <!-- Wheel Information -->
-            <left_joint>base_left_wheel_joint</left_joint>
-            <right_joint>base_right_wheel_joint</right_joint>
+            <left_joint>left_wheel_joint</left_joint>
+            <right_joint>right_wheel_joint</right_joint>
             <topic>cmd_vel</topic>
-            <!-- <odom_topic>odom</odom_topic>
             <frame_id>odom</frame_id>
-            <child_frame_id>base_footprint</child_frame_id> -->
-            <wheel_separation>0.45</wheel_separation>
-            <wheel_radius>0.1</wheel_radius>
+            <child_frame_id>base_link</child_frame_id>
+            <wheel_separation>0.297</wheel_separation>
+            <wheel_radius>0.066</wheel_radius>
             <odom_publish_frequency>100</odom_publish_frequency>
-            <max_linear_acceleration>1</max_linear_acceleration>
-            <min_linear_acceleration>-1</min_linear_acceleration>
-            <max_angular_acceleration>2</max_angular_acceleration>
-            <min_angular_acceleration>-2</min_angular_acceleration>
-            <max_linear_velocity>0.5</max_linear_velocity>
-            <min_linear_velocity>-0.5</min_linear_velocity>
-            <max_angular_velocity>1</max_angular_velocity>
-            <min_angular_velocity>-1</min_angular_velocity>
+            <publish_odom>true</publish_odom>
         </plugin>
         <plugin filename="ignition-gazebo-odometry-publisher-system"
                 name="ignition::gazebo::systems::OdometryPublisher">
             <odom_frame>odom</odom_frame>
-            <odom_covariance_topic>odom</odom_covariance_topic>
+            <!-- <odom_covariance_topic>odom</odom_covariance_topic> -->
             <tf_topic>tf</tf_topic>
             <robot_base_frame>base_link</robot_base_frame>
             <odom_publish_frequency>100</odom_publish_frequency>
         </plugin>
-        <!-- <plugin filename="ignition-gazebo-velocity-control-system"
-                name="ignition::gazebo::systems::VelocityControl">
-            <topic>cmd_vel</topic>
-        </plugin> -->
+        <plugin filename="ignition-gazebo-pose-publisher-system" name="ignition::gazebo::systems::PosePublisher">
+            <publish_link_pose>true</publish_link_pose>
+            <publish_collision_pose>false</publish_collision_pose>
+            <publish_visual_pose>false</publish_visual_pose>
+            <publish_sensor_pose>false</publish_sensor_pose>
+            <publish_nested_model_pose>true</publish_nested_model_pose>
+            <update_frequency>20</update_frequency>
+        </plugin>
     </gazebo>
 </robot>

File: src/testbot/description/lidar.xacro (robot description, xacro)
@@ -2,29 +2,10 @@
 <robot xmlns:xacro="http://www.ros.org/wiki/xacro">
     <!-- INITIATE GAZEBO LIDAR SENSOR -->
-    <link name="lidar_link">
-        <visual>
-            <geometry>
-                <cylinder radius="0.09" length="0.05" />
-            </geometry>
-            <origin xyz="0 0 0" rpy="0 0 0" />
-            <material name="white" />
-        </visual>
-        <collision>
-            <geometry>
-                <box size ="0.18 0.18 0.05" />
-            </geometry>
-            <origin xyz="0 0 0" rpy="0 0 0" />
-        </collision>
-    </link>
-    <joint name="base_laser_joint" type="fixed">
-        <parent link="base_link"/>
-        <child link="lidar_link"/>
-        <origin xyz="0 0 0.225" rpy="0 0 0"/>
-    </joint>
     <gazebo reference="lidar_link">
         <sensor name="lidar_sensor" type="gpu_lidar">
-            <topic>LaserScan</topic>
+            <ignition_frame_id>lidar_link</ignition_frame_id>
+            <topic>scan</topic>
             <pose>0 0 0 0 0 0</pose>
-            <update_rate>5</update_rate>
+            <update_rate>10</update_rate>
             <ray>
                 <scan>
@@ -39,5 +20,5 @@
                     <min>0.3</min>
                     <max>12</max>
-                    <resolution>0.01</resolution>
+                    <resolution>1</resolution>
                 </range>
             </ray>

File: src/testbot/description/test_robot.urdf.xacro (robot description, xacro)
@@ -1,5 +1,5 @@
 <?xml version="1.0"?>
 <robot name="test_robot" xmlns:xacro="http://www.ros.org/wiki/xacro">
-    <xacro:include filename="test_robot_core.xacro" />
+    <xacro:include filename="test_robot_core2.xacro" />
     <!-- <xacro:include filename="ros2_control.xacro" /> -->
     <xacro:include filename="gazebo_control.xacro" />

File: src/testbot/description/test_robot_core2.xacro (robot description, xacro)
@@ -1,6 +1,19 @@
 <?xml version="1.0"?>
 <robot xmlns:xacro="http://www.ros.org/wiki/xacro">
-#Include connected files
-    <xacro:include filename="inertial_macros.xacro" />
+    <xacro:include filename="inertial_macros.xacro"/>
+    <xacro:property name="chassis_length" value="0.335"/>
+    <xacro:property name="chassis_width" value="0.265"/>
+    <xacro:property name="chassis_height" value="0.138"/>
+    <xacro:property name="chassis_mass" value="1.0"/>
+    <xacro:property name="wheel_radius" value="0.033"/>
+    <xacro:property name="wheel_thickness" value="0.026"/>
+    <xacro:property name="wheel_mass" value="0.05"/>
+    <xacro:property name="wheel_offset_x" value="0.226"/>
+    <xacro:property name="wheel_offset_y" value="0.1485"/>
+    <xacro:property name="wheel_offset_z" value="0.01"/>
+    <xacro:property name="caster_wheel_radius" value="0.01"/>
+    <xacro:property name="caster_wheel_mass" value="0.01"/>
+    <xacro:property name="caster_wheel_offset_x" value="0.075"/>
+    <xacro:property name="caster_wheel_offset_z" value="${wheel_offset_z - wheel_radius + caster_wheel_radius}"/>
 #Define colours
     <material name="grey">
@@ -13,137 +26,142 @@
         <color rgba ="1 1 1 1" />
     </material>
-#LINKS
-    <!-- ROBOT FOOTPRINT LINK -->
-    <link name="base_footprint" />
-    <!-- ROBOT BODY LINK -->
+    <!-- BASE LINK -->
     <link name="base_link">
+    </link>
+    <!-- BASE_FOOTPRINT LINK -->
+    <joint name="base_footprint_joint" type="fixed">
+        <parent link="base_link"/>
+        <child link="base_footprint"/>
+        <origin xyz="0 0 0" rpy="0 0 0"/>
+    </joint>
+    <link name="base_footprint">
+    </link>
+    <!-- CHASSIS LINK -->
+    <joint name="chassis_joint" type="fixed">
+        <parent link="base_link"/>
+        <child link="chassis"/>
+        <origin xyz="${-wheel_offset_x} 0 ${-wheel_offset_z + wheel_radius}"/>
+    </joint>
+    <link name="chassis">
+        <visual>
+            <origin xyz="${chassis_length/2} 0 ${chassis_height/2}"/>
+            <geometry>
+                <box size="${chassis_length} ${chassis_width} ${chassis_height}"/>
+            </geometry>
+            <material name="purple"/>
+        </visual>
+        <collision>
+            <origin xyz="${chassis_length/2} 0 ${chassis_height/2}"/>
+            <geometry>
+                <box size="${chassis_length} ${chassis_width} ${chassis_height}"/>
+            </geometry>
+        </collision>
+        <xacro:inertial_box mass="0.5" x="${chassis_length}" y="${chassis_width}" z="${chassis_height}">
+            <origin xyz="${chassis_length/2} 0 ${chassis_height/2}" rpy="0 0 0"/>
+        </xacro:inertial_box>
+    </link>
+    <!-- LEFT WHEEL LINK -->
+    <joint name="left_wheel_joint" type="continuous">
+        <parent link="base_link"/>
+        <child link="left_wheel"/>
+        <origin xyz="0 ${wheel_offset_y} ${wheel_radius}" rpy="-${pi/2} 0 0" />
+        <axis xyz="0 0 1"/>
+    </joint>
+    <link name="left_wheel">
         <visual>
             <geometry>
-                <box size ="0.6 0.4 0.2" />
+                <cylinder radius="${wheel_radius}" length="${wheel_thickness}"/>
             </geometry>
-            <origin xyz="0 0 0.1" rpy="0 0 0" />
-            <material name="purple" />
+            <material name="grey"/>
         </visual>
         <collision>
             <geometry>
-                <box size ="0.6 0.4 0.2" />
+                <sphere radius="${wheel_radius}"/>
             </geometry>
-            <origin xyz="0 0 0.1" rpy="0 0 0" />
         </collision>
-        <xacro:inertial_box mass="0.5" x="0.6" y="0.4" z="0.2">
-            <origin xyz="0 0 0.1" rpy="0 0 0" />
-        </xacro:inertial_box>
+        <xacro:inertial_cylinder mass="${wheel_mass}" length="${wheel_thickness}" radius="${wheel_radius}">
+            <origin xyz="0 0 0" rpy="0 0 0"/>
+        </xacro:inertial_cylinder>
     </link>
-    <!-- LIDAR LINK -->
-    <link name="lidar_module">
+    <!-- RIGHT WHEEL LINK -->
+    <joint name="right_wheel_joint" type="continuous">
+        <parent link="base_link"/>
+        <child link="right_wheel"/>
+        <origin xyz="0 ${-wheel_offset_y} ${wheel_radius}" rpy="${pi/2} 0 0" />
+        <axis xyz="0 0 -1"/>
+    </joint>
+    <link name="right_wheel">
         <visual>
             <geometry>
-                <cylinder radius="0.09" length="0.05" />
+                <cylinder radius="${wheel_radius}" length="${wheel_thickness}"/>
             </geometry>
-            <origin xyz="0 0 0" rpy="0 0 0" />
-            <material name="white" />
+            <material name="grey"/>
         </visual>
         <collision>
             <geometry>
-                <box size ="0.18 0.18 0.05" />
+                <sphere radius="${wheel_radius}"/>
             </geometry>
-            <origin xyz="0 0 0" rpy="0 0 0" />
         </collision>
+        <xacro:inertial_cylinder mass="${wheel_mass}" length="${wheel_thickness}" radius="${wheel_radius}">
+            <origin xyz="0 0 0" rpy="0 0 0"/>
+        </xacro:inertial_cylinder>
     </link>
-    <!-- LEFT WHEEL LINK -->
-    <link name="left_wheel">
+    <gazebo reference="right_wheel">
+        <material>Gazebo/Blue</material>
+    </gazebo>
+    <!-- CASTER WHEEL LINK -->
+    <joint name="caster_wheel_joint" type="fixed">
+        <parent link="chassis"/>
+        <child link="caster_wheel"/>
+        <origin xyz="${caster_wheel_offset_x} 0 ${caster_wheel_offset_z}"/>
+    </joint>
+    <link name="caster_wheel">
         <visual>
             <geometry>
-                <cylinder radius="0.1" length="0.05" />
+                <sphere radius="${caster_wheel_radius}"/>
             </geometry>
-            <origin xyz="0 0.025 0" rpy="1.57 0 0" />
-            <material name="grey" />
+            <material name="grey"/>
         </visual>
         <collision>
             <geometry>
-                <!-- use sphere collider for minimal contact with ground to eliminate wheel drift -->
-                <sphere radius ="0.1" />
+                <sphere radius="${caster_wheel_radius}"/>
             </geometry>
-            <origin xyz="0 0.025 0" rpy="1.57 0 0" />
         </collision>
-        <xacro:inertial_cylinder mass="0.1" radius="0.1" length="0.05">
-            <origin xyz="0 0.025 0" rpy="1.57 0 0" />
-        </xacro:inertial_cylinder>
+        <xacro:inertial_sphere mass="${caster_wheel_mass}" radius="${caster_wheel_radius}">
+            <origin xyz="0 0 0" rpy="0 0 0"/>
+        </xacro:inertial_sphere>
     </link>
-    <!-- RIGHT WHEEL LINK -->
-    <link name="right_wheel">
+    <gazebo reference="caster_wheel">
+        <mu1 value="0.001"/>
+        <mu2 value="0.001"/>
+    </gazebo>
+    <!-- LIDAR LINK -->
+    <joint name="lidar_joint" type="fixed">
+        <parent link="chassis"/>
+        <child link="lidar_link"/>
+        <origin xyz="0.122 0 0.212" rpy="0 0 0"/>
+    </joint>
+    <link name="lidar_link">
         <visual>
             <geometry>
-                <cylinder radius="0.1" length="0.05" />
+                <cylinder radius="0.05" length="0.04"/>
             </geometry>
-            <origin xyz="0 -0.025 0" rpy="-1.57 0 0" />
-            <material name="grey" />
+            <material name="white"/>
+        </visual>
+        <visual>
+            <origin xyz="0 0 -0.05"/>
+            <geometry>
+                <cylinder radius="0.01" length="0.1"/>
+            </geometry>
+            <material name="white"/>
         </visual>
         <collision>
             <geometry>
-                <!-- use sphere colliders for minimal contact with ground to eliminate wheel drift -->
-                <sphere radius="0.1" />
+                <cylinder radius="0.05" length="0.04"/>
             </geometry>
-            <origin xyz="0 -0.025 0" rpy="-1.57 0 0" />
         </collision>
-        <xacro:inertial_cylinder mass="0.1" radius="0.1" length="0.05">
-            <origin xyz="0 -0.025 0" rpy="-1.57 0 0" />
+        <xacro:inertial_cylinder mass="0.1" length="0.04" radius="0.05">
+            <origin xyz="0 0 0" rpy="0 0 0"/>
         </xacro:inertial_cylinder>
     </link>
-    <!-- CASTER WHEEL LINK -->
-    <link name="caster_wheel">
-        <visual>
-            <geometry>
-                <sphere radius="0.05" />
-            </geometry>
-            <origin xyz="0 0 -0.05" rpy="0 0 0" />
-            <material name="grey" />
-        </visual>
-        <collision>
-            <geometry>
-                <sphere radius="0.05" />
-            </geometry>
-            <origin xyz="0 0 -0.05" rpy="0 0 0" />
-        </collision>
-        <xacro:inertial_sphere mass="0.08" radius="0.05">
-            <origin xyz="0 0 -0.05" rpy="0 0 0" />
-        </xacro:inertial_sphere>
-    </link>
-    <gazebo reference="caster_wheel">
-        <mu1 value ="0.001"/>
-        <mu2 value ="0.001"/>
-    </gazebo>
-#JOINTS
-    <!-- ROBOT BODY FOOTPRINT JOINT -->
-    <joint name="base_joint" type="fixed">
-        <parent link="base_footprint" />
-        <child link="base_link" />
-        <origin xyz="0 0 0.1" rpy="0 0 0" />
-    </joint>
-    <!-- LIDAR JOINT -->
-    <joint name="base_lidar_module_joint" type="fixed">
-        <parent link="base_link" />
-        <child link="lidar_module" />
-        <origin xyz="0 0 0.225" rpy="0 0 0" />
-    </joint>
-    <!-- LEFT WHEEL JOINT -->
-    <joint name="base_left_wheel_joint" type="continuous">
-        <parent link="base_link" />
-        <child link="left_wheel" />
-        <origin xyz="-0.15 0.2 0" rpy="0 0 0" />
-        <axis xyz="0 1 0" />
-    </joint>
-    <!-- RIGHT WHEEL JOINT -->
-    <joint name="base_right_wheel_joint" type="continuous">
-        <parent link="base_link" />
-        <child link="right_wheel" />
-        <origin xyz="-0.15 -0.2 0" rpy="0 0 0" />
-        <axis xyz="0 1 0" />
-    </joint>
-    <!-- CASTER WHEEL JOINT -->
-    <joint name="base_caster_wheel_joint" type="fixed">
-        <parent link="base_link" />
-        <child link="caster_wheel" />
-        <origin xyz="0.2 0 0" rpy="0 0 0" />
-    </joint>
 </robot>
